File: eda/altbier_pcb_3d6/altbier_pcb_3d6.kicad_pcb (KiCad board)
At the start: 2 copper layers, 0 parts

Commit message: schematic rework with new button
Parts:
- added C1: 0.1uF/100nF, 0_local:C_0805_2012Metric, F.Cu at (81.2, 92.5)
- added C2: 0.1uF/100nF, 0_local:C_0805_2012Metric, F.Cu at (80.5, 98.3)
- added D11: Red, 0_local:LED_0805_2012Metric, F.Cu at (115.0, 75.2)
- added D12: Red, 0_local:LED_0805_2012Metric, F.Cu at (125.0, 85.0)
- added D13: Red, 0_local:LED_0805_2012Metric, F.Cu at (114.9, 80.0)
- added D14: Red, 0_local:LED_0805_2012Metric, F.Cu at (125.0, 80.0)
- added D15: Red, 0_local:LED_0805_2012Metric, F.Cu at (114.8, 85.0)
- added D16: Red, 0_local:LED_0805_2012Metric, F.Cu at (125.0, 75.0)
- added D17: Red, 0_local:LED_0805_2012Metric, F.Cu at (120.0, 80.0)
- added D21: Green, 0_local:LED_0805_2012Metric, F.Cu at (155.0, 75.0)
- added D22: Green, 0_local:LED_0805_2012Metric, F.Cu at (165.0, 85.0)
- added D23: Green, 0_local:LED_0805_2012Metric, F.Cu at (155.0, 80.0)
- added D24: Green, 0_local:LED_0805_2012Metric, F.Cu at (165.0, 80.0)
- added D25: Green, 0_local:LED_0805_2012Metric, F.Cu at (154.9, 85.0)
- added D26: Green, 0_local:LED_0805_2012Metric, F.Cu at (165.0, 75.0)
- added D27: Green, 0_local:LED_0805_2012Metric, F.Cu at (160.0, 80.0)
- added D31: Blue, 0_local:LED_0805_2012Metric, F.Cu at (195.0, 75.0)
- added D32: Blue, 0_local:LED_0805_2012Metric, F.Cu at (205.0, 85.0)
- added D33: Blue, 0_local:LED_0805_2012Metric, F.Cu at (195.0, 80.0)
- added D34: Blue, 0_local:LED_0805_2012Metric, F.Cu at (205.0, 80.0)
- added D35: Blue, 0_local:LED_0805_2012Metric, F.Cu at (195.0, 85.0)
- added D36: Blue, 0_local:LED_0805_2012Metric, F.Cu at (205.0, 75.0)
- added D37: Blue, 0_local:LED_0805_2012Metric, F.Cu at (200.0, 80.0)
- added IC1: IC_CH552G, 0_local:IC_SOIC-16_3.9x9.9mm_Pitch1.27mm, F.Cu at (95.0, 110.0)
- added J1: USB_B_Micro, 0_local:USB_Micro-B_Jing, F.Cu at (65.0, 140.0)
- added J2: Conn_01x02, 0_local:Conn_Pin_Header_Straight_1x02_Pitch2.54mm, F.Cu at (70.0, 110.0)
- added R11: 200 Ohms, 0_local:R_0805_2012Metric, F.Cu at (105.0, 95.0)
- added R12: 200 Ohms, 0_local:R_0805_2012Metric, F.Cu at (125.0, 95.0)
- added R13: 200 Ohms, 0_local:R_0805_2012Metric, F.Cu at (110.0, 95.0)
- added R14: 200 Ohms, 0_local:R_0805_2012Metric, F.Cu at (130.0, 95.0)
- added R15: 200 Ohms, 0_local:R_0805_2012Metric, F.Cu at (115.0, 95.0)
- added R16: 200 Ohms, 0_local:R_0805_2012Metric, F.Cu at (135.0, 95.0)
- added R17: 200 Ohms, 0_local:R_0805_2012Metric, F.Cu at (120.0, 95.0)
- added R2: 10k Ohms, 0_local:R_0805_2012Metric, F.Cu at (65.9, 150.0)
- added R21: 200 Ohms, 0_local:R_0805_2012Metric, F.Cu at (145.0, 95.0)
- added R22: 200 Ohms, 0_local:R_0805_2012Metric, F.Cu at (165.0, 95.0)
- added R23: 200 Ohms, 0_local:R_0805_2012Metric, F.Cu at (150.0, 95.0)
- added R24: 200 Ohms, 0_local:R_0805_2012Metric, F.Cu at (170.0, 95.0)
- added R25: 200 Ohms, 0_local:R_0805_2012Metric, F.Cu at (155.0, 95.0)
- added R26: 200 Ohms, 0_local:R_0805_2012Metric, F.Cu at (175.0, 95.0)
- added R27: 200 Ohms, 0_local:R_0805_2012Metric, F.Cu at (160.0, 95.0)
- added R3: 10k Ohms, 0_local:R_0805_2012Metric, F.Cu at (139.6, 120.4)
- added R31: 200 Ohms, 0_local:R_0805_2012Metric, F.Cu at (185.0, 95.0)
- added R32: 200 Ohms, 0_local:R_0805_2012Metric, F.Cu at (205.0, 95.0)
- added R33: 200 Ohms, 0_local:R_0805_2012Metric, F.Cu at (190.0, 95.0)
- added R34: 200 Ohms, 0_local:R_0805_2012Metric, F.Cu at (210.0, 95.0)
- added R35: 200 Ohms, 0_local:R_0805_2012Metric, F.Cu at (195.0, 95.0)
- added R36: 200 Ohms, 0_local:R_0805_2012Metric, F.Cu at (215.0, 95.0)
- added R37: 200 Ohms, 0_local:R_0805_2012Metric, F.Cu at (200.0, 95.0)
- added SW1: SPDT_C136659, 0_local:SW_SPDT_PCM12_C136659, F.Cu at (65.0, 125.0)
- added SW2: TS2306A, 0_local:SW_TS2306A240GFMSM9_C388290, F.Cu at (66.4, 160.0)
- added SW3: SW_Push_SPST_4pin, 0_local:SW_TS3735PA250GF, F.Cu at (131.4, 115.5)
